Commit message: 修复了urdf、robot_start.launch,还有部分功能包的cmake和package文件

File: src/robot_description/urdf/robot_description.urdf (robot description, URDF)
Before this commit: robot robot_description, 15 links, 14 joints
Links:
- removed link rader_link
- added link laser_frame, mass 0.0197577859576288; collision mesh filename=package://robot_description/meshes/rader_link.STL; visual mesh filename=package://robot_description/meshes/rader_link.STL
Joints:
- removed joint rader
- added joint laser_joint: type fixed, parent base_link, child laser_frame, origin xyz=-0.000482541160108889 0 0.111874126705049 rpy=0 0 0, axis 0 0 0
- joint arm1: limit lower=-210 upper=0 effort=1 velocity=3 -> lower=-3.66519 upper=0 effort=1 velocity=3
- joint arm2: limit lower=0 upper=270 effort=1 velocity=3 -> lower=0 upper=3.66519 effort=1 velocity=3
- joint arm3: limit lower=0 upper=100 effort=1 velocity=3 -> lower=0 upper=1.74533 effort=1 velocity=3
- joint arm4: limit lower=-90 upper=90 effort=1 velocity=3 -> lower=-1.5708 upper=1.5708 effort=1 velocity=3

Commit message: 测试并使robot_description功能包正常工作

File: src/robot_description/urdf/robot_description.urdf (robot description, URDF)
Before this commit: robot robot_description, 15 links, 14 joints
Links:
- added link base_footprint
- link LFd_Link: mass 0.0555886189628007 -> 0.0555886189628006
- link LFs_Link: mass 0.114715980474315 -> 0.114715980836134
- link RFd_Link: mass 0.0555886189628006 -> 0.0555886189628007
- link arm1_Link: mass 0.190587416523155 -> 0.1905874165244
- link arm2_Link: mass 0.164248712945773 -> 0.164248712945774
- link arm3_Link: mass 0.0312238812156414 -> 0.0312238812156817
- link arm4_Link: mass 0.0522475609220887 -> 0.0522475609584348
- link base_link: mass 3.02079029985786 -> 3.02079030126272
- link laser_frame: geometry collision mesh filename=package://robot_description/meshes/laser_frame.STL; visual mesh filename=package://robot_description/meshes/laser_frame.STL
Joints:
- removed joint laser_joint
- added joint base_joint: type fixed, parent base_footprint, child base_link, origin xyz=0.0 0.0 0.033 rpy=0 0 0
- added joint laser_frame_joint: type fixed, parent base_link, child laser_frame, origin xyz=-0.000482541160108889 0 0.111874126705049 rpy=0 0 0, axis 0 0 0
- joint LRd: origin xyz=0.265730891387391 -0.0192000149036779 -0.05495771030536 rpy=1.5707963267949 0 0 -> xyz=0 -0.0192000149011577 -0.0549577103053588 rpy=1.5707963267949 0 0
- joint arm0: origin xyz=0.029517 0 0.17312 rpy=0 0 0 -> xyz=0.0295174588398881 0 0.173124126705049 rpy=0 0 0
- joint arm1: limit lower=-3.66519 upper=0 effort=1 velocity=3 -> lower=-210 upper=0 effort=1 velocity=3
- joint arm2: limit lower=0 upper=3.66519 effort=1 velocity=3 -> lower=0 upper=270 effort=1 velocity=3; origin xyz=-0.2143 0 0.0376 rpy=0 0 0 -> xyz=-0.214299994813131 0 0.0376000028997485 rpy=0 0 0
- joint arm3: axis -0.0087259 -0.0087265 -0.99992 -> -0.00872587097686232 -0.00872653549837341 -0.99992385047757; limit lower=0 upper=1.74533 effort=1 velocity=3 -> lower=0 upper=100 effort=1 velocity=3; origin xyz=0.1952 0.047998 0.00049999 rpy=0.008727 -0.008726 -7.6152E-05 -> xyz=0.195198405547995 0.0479983915101106 0.000499985962073995 rpy=0.00872697851439958 -0.00872598171315928 -7.61524215215586E-05
- joint arm4: axis -0.0087259 -0.0087265 -0.99992 -> -0.00872587097688493 -0.00872653523448956 -0.999923850479873; limit lower=-1.5708 upper=1.5708 effort=1 velocity=3 -> lower=-90 upper=90 effort=1 velocity=3; origin xyz=0.039893 -0.034669 -0.018347 rpy=1.5682 0.0050959 -0.36648 -> xyz=0.0398926340613602 -0.0346685199789408 -0.0183469477877459 rpy=1.56824861064815 0.00509594419856987 -0.366478515653153

Commit message: 修改urdf雷达命名，nav2配置文件

File: src/robot_description/urdf/robot_description.urdf (robot description, URDF)
Before this commit: robot robot_description, 16 links, 15 joints
Links:
- removed link laser_frame
- added link laser, mass 0.0197577859576288; collision mesh filename=package://robot_description/meshes/laser_frame.STL; visual mesh filename=package://robot_description/meshes/laser_frame.STL
Joints:
- removed joint laser_frame_joint
- added joint laser_joint: type fixed, parent base_link, child laser, origin xyz=-0.000482541160108889 0 0.111874126705049 rpy=0 0 0, axis 0 0 0
