Commit message: feat: add Gazebo plugins to robot_sim.xacro
- Simplified collision geometry (box/cylinder)
- Planar move plugin for cmd_vel control
- Joint state publisher for /joint_states
- Ray sensor for 2D LiDAR /scan

Co-Authored-By: Claude Opus 4.8 <noreply@anthropic.com>

File: src/robot_gazebo/urdf/robot_sim.xacro (robot description, xacro)
@@ -461,6 +461,190 @@
   </joint>
   <!-- ================================================================
-       Gazebo plugin tags — see Task 3
+       Gazebo Simulation Plugins
        ================================================================ -->
-  <!-- PLACEHOLDER: Task 3 will insert gazebo plugins here -->
+  <!-- ===== Collision Overrides (simplified geometry) ===== -->
+  <gazebo reference="base_link">
+    <collision>
+      <geometry>
+        <box>
+          <size>0.6 0.5 0.25</size>
+        </box>
+      </geometry>
+    </collision>
+    <maxContacts>10</maxContacts>
+  </gazebo>
+  <gazebo reference="laser">
+    <collision>
+      <geometry>
+        <box>
+          <size>0.07 0.07 0.07</size>
+        </box>
+      </geometry>
+    </collision>
+  </gazebo>
+  <!-- Steering links: LFs, LRs, RFs, RRs -->
+  <gazebo reference="LFs_Link">
+    <collision>
+      <geometry>
+        <cylinder radius="0.02" length="0.04"/>
+      </geometry>
+    </collision>
+  </gazebo>
+  <gazebo reference="LRs_Link">
+    <collision>
+      <geometry>
+        <cylinder radius="0.02" length="0.04"/>
+      </geometry>
+    </collision>
+  </gazebo>
+  <gazebo reference="RFs_Link">
+    <collision>
+      <geometry>
+        <cylinder radius="0.02" length="0.04"/>
+      </geometry>
+    </collision>
+  </gazebo>
+  <gazebo reference="RRs_Link">
+    <collision>
+      <geometry>
+        <cylinder radius="0.02" length="0.04"/>
+      </geometry>
+    </collision>
+  </gazebo>
+  <!-- Drive links: LFd, LRd, RFd, RRd -->
+  <gazebo reference="LFd_Link">
+    <collision>
+      <geometry>
+        <cylinder radius="0.033" length="0.02"/>
+      </geometry>
+    </collision>
+    <material>
+      <uri>model://grey</uri>
+    </material>
+  </gazebo>
+  <gazebo reference="LRd_Link">
+    <collision>
+      <geometry>
+        <cylinder radius="0.033" length="0.02"/>
+      </geometry>
+    </collision>
+  </gazebo>
+  <gazebo reference="RFd_Link">
+    <collision>
+      <geometry>
+        <cylinder radius="0.033" length="0.02"/>
+      </geometry>
+    </collision>
+  </gazebo>
+  <gazebo reference="RRd_Link">
+    <collision>
+      <geometry>
+        <cylinder radius="0.033" length="0.02"/>
+      </geometry>
+    </collision>
+  </gazebo>
+  <!-- Arm links: disable collision (not simulated) -->
+  <gazebo reference="arm0_Link">
+    <collision>
+      <geometry>
+        <box>
+          <size>0.01 0.01 0.01</size>
+        </box>
+      </geometry>
+    </collision>
+  </gazebo>
+  <gazebo reference="arm1_Link">
+    <collision>
+      <geometry>
+        <box>
+          <size>0.01 0.01 0.01</size>
+        </box>
+      </geometry>
+    </collision>
+  </gazebo>
+  <gazebo reference="arm2_Link">
+    <collision>
+      <geometry>
+        <box>
+          <size>0.01 0.01 0.01</size>
+        </box>
+      </geometry>
+    </collision>
+  </gazebo>
+  <gazebo reference="arm3_Link">
+    <collision>
+      <geometry>
+        <box>
+          <size>0.01 0.01 0.01</size>
+        </box>
+      </geometry>
+    </collision>
+  </gazebo>
+  <gazebo reference="arm4_Link">
+    <collision>
+      <geometry>
+        <box>
+          <size>0.01 0.01 0.01</size>
+        </box>
+      </geometry>
+    </collision>
+  </gazebo>
+  <!-- ===== Planar Move Plugin (cmd_vel → base motion + odom) ===== -->
+  <gazebo>
+    <plugin name="planar_move" filename="libgazebo_ros_planar_move.so">
+      <ros>
+        <namespace>/</namespace>
+      </ros>
+      <command_topic>cmd_vel</command_topic>
+      <odometry_topic>odom</odometry_topic>
+      <odometry_frame>odom</odometry_frame>
+      <robot_base_frame>base_footprint</robot_base_frame>
+      <publish_odom_tf>true</publish_odom_tf>
+      <odometry_publish_rate>30.0</odometry_publish_rate>
+    </plugin>
+  </gazebo>
+  <!-- ===== Joint State Publisher (→ /joint_states) ===== -->
+  <gazebo>
+    <plugin name="joint_state_publisher" filename="libgazebo_ros_joint_state_publisher.so">
+      <ros>
+        <namespace>/</namespace>
+        <remapping>~/out:=joint_states</remapping>
+      </ros>
+      <update_rate>30</update_rate>
+    </plugin>
+  </gazebo>
+  <!-- ===== 2D LiDAR Ray Sensor (→ /scan) ===== -->
+  <gazebo reference="laser">
+    <sensor type="ray" name="laser_sensor">
+      <pose>0 0 0 0 0 0</pose>
+      <visualize>false</visualize>
+      <update_rate>10</update_rate>
+      <ray>
+        <scan>
+          <horizontal>
+            <samples>360</samples>
+            <resolution>1</resolution>
+            <min_angle>-3.14159</min_angle>
+            <max_angle>3.14159</max_angle>
+          </horizontal>
+        </scan>
+        <range>
+          <min>0.15</min>
+          <max>30.0</max>
+        </range>
+        <noise>
+          <type>gaussian</type>
+          <mean>0.0</mean>
+          <stddev>0.01</stddev>
+        </noise>
+      </ray>
+      <plugin name="laser_controller" filename="libgazebo_ros_ray_sensor.so">
+        <ros>
+          <namespace>/</namespace>
+          <remapping>~/out:=scan</remapping>
+        </ros>
+        <frame_name>laser</frame_name>
+      </plugin>
+    </sensor>
+  </gazebo>
 </robot>

Commit message: fix: correct planar_move plugin parameters and sensor config
- Use correct gazebo_plugins planar_move API (update_rate, publish_rate, publish_odom)
- Remove invalid command_topic/odometry_topic (use ros defaults)
- Replace odometry_publish_rate with publish_rate
- Add output_type sensor_msgs/LaserScan to ray sensor
- Remove inconsistent material tag from single drive wheel (LFd_Link)

Co-Authored-By: Claude Opus 4.8 <noreply@anthropic.com>

File: src/robot_gazebo/urdf/robot_sim.xacro (robot description, xacro)
@@ -519,7 +519,4 @@
       </geometry>
     </collision>
-    <material>
-      <uri>model://grey</uri>
-    </material>
   </gazebo>
   <gazebo reference="LRd_Link">
@@ -596,10 +593,10 @@
         <namespace>/</namespace>
       </ros>
-      <command_topic>cmd_vel</command_topic>
-      <odometry_topic>odom</odometry_topic>
+      <update_rate>100.0</update_rate>
+      <publish_rate>30.0</publish_rate>
+      <publish_odom>true</publish_odom>
+      <publish_odom_tf>true</publish_odom_tf>
       <odometry_frame>odom</odometry_frame>
       <robot_base_frame>base_footprint</robot_base_frame>
-      <publish_odom_tf>true</publish_odom_tf>
-      <odometry_publish_rate>30.0</odometry_publish_rate>
     </plugin>
   </gazebo>
@@ -644,4 +641,5 @@
           <remapping>~/out:=scan</remapping>
         </ros>
+        <output_type>sensor_msgs/LaserScan</output_type>
         <frame_name>laser</frame_name>
       </plugin>

Commit message: fix: cylinder SDF format and world_path CLI argument
- Change cylinder collision from URDF attribute style (radius=, length=)
  to SDF child-element style (<radius>, <length>) to fix Gazebo warnings:
  'XML Attribute[radius] in element[cylinder] not defined in SDF, ignoring'
- Add DeclareLaunchArgument for world_path so users can override
  the world file from command line

Co-Authored-By: Claude Opus 4.8 <noreply@anthropic.com>

File: src/robot_gazebo/urdf/robot_sim.xacro (robot description, xacro)
@@ -487,5 +487,8 @@
     <collision>
       <geometry>
-        <cylinder radius="0.02" length="0.04"/>
+        <cylinder>
+          <radius>0.02</radius>
+          <length>0.04</length>
+        </cylinder>
       </geometry>
     </collision>
@@ -494,5 +497,8 @@
     <collision>
       <geometry>
-        <cylinder radius="0.02" length="0.04"/>
+        <cylinder>
+          <radius>0.02</radius>
+          <length>0.04</length>
+        </cylinder>
       </geometry>
     </collision>
@@ -501,5 +507,8 @@
     <collision>
       <geometry>
-        <cylinder radius="0.02" length="0.04"/>
+        <cylinder>
+          <radius>0.02</radius>
+          <length>0.04</length>
+        </cylinder>
       </geometry>
     </collision>
@@ -508,5 +517,8 @@
     <collision>
       <geometry>
-        <cylinder radius="0.02" length="0.04"/>
+        <cylinder>
+          <radius>0.02</radius>
+          <length>0.04</length>
+        </cylinder>
       </geometry>
     </collision>
@@ -516,5 +528,8 @@
     <collision>
       <geometry>
-        <cylinder radius="0.033" length="0.02"/>
+        <cylinder>
+          <radius>0.033</radius>
+          <length>0.02</length>
+        </cylinder>
       </geometry>
     </collision>
@@ -523,5 +538,8 @@
     <collision>
       <geometry>
-        <cylinder radius="0.033" length="0.02"/>
+        <cylinder>
+          <radius>0.033</radius>
+          <length>0.02</length>
+        </cylinder>
       </geometry>
     </collision>
@@ -530,5 +548,8 @@
     <collision>
       <geometry>
-        <cylinder radius="0.033" length="0.02"/>
+        <cylinder>
+          <radius>0.033</radius>
+          <length>0.02</length>
+        </cylinder>
       </geometry>
     </collision>
@@ -537,5 +558,8 @@
     <collision>
       <geometry>
-        <cylinder radius="0.033" length="0.02"/>
+        <cylinder>
+          <radius>0.033</radius>
+          <length>0.02</length>
+        </cylinder>
       </geometry>
     </collision>
