Commit message: 搭建gazebo仿真

File: src/robot_gazebo/urdf/robot_sim.xacro (robot description, xacro)
@@ -23,5 +23,5 @@
       <origin xyz="0 0 0" rpy="0 0 0"/>
       <geometry>
-        <mesh filename="package://robot_description/meshes/base_link.STL"/>
+        <mesh filename="$(find robot_description)/meshes/base_link.STL"/>
       </geometry>
       <material name="">
@@ -32,5 +32,5 @@
       <origin xyz="0 0 0" rpy="0 0 0"/>
       <geometry>
-        <mesh filename="package://robot_description/meshes/base_link.STL"/>
+        <mesh filename="$(find robot_description)/meshes/base_link.STL"/>
       </geometry>
     </collision>
@@ -46,5 +46,5 @@
       <origin xyz="0 0 0" rpy="0 0 0"/>
       <geometry>
-        <mesh filename="package://robot_description/meshes/laser_frame.STL"/>
+        <mesh filename="$(find robot_description)/meshes/laser_frame.STL"/>
       </geometry>
       <material name="">
@@ -55,5 +55,5 @@
       <origin xyz="0 0 0" rpy="0 0 0"/>
       <geometry>
-        <mesh filename="package://robot_description/meshes/laser_frame.STL"/>
+        <mesh filename="$(find robot_description)/meshes/laser_frame.STL"/>
       </geometry>
     </collision>
@@ -76,5 +76,5 @@
       <origin xyz="0 0 0" rpy="0 0 0"/>
       <geometry>
-        <mesh filename="package://robot_description/meshes/arm0_Link.STL"/>
+        <mesh filename="$(find robot_description)/meshes/arm0_Link.STL"/>
       </geometry>
       <material name="">
@@ -85,5 +85,5 @@
       <origin xyz="0 0 0" rpy="0 0 0"/>
       <geometry>
-        <mesh filename="package://robot_description/meshes/arm0_Link.STL"/>
+        <mesh filename="$(find robot_description)/meshes/arm0_Link.STL"/>
       </geometry>
     </collision>
@@ -106,5 +106,5 @@
       <origin xyz="0 0 0" rpy="0 0 0"/>
       <geometry>
-        <mesh filename="package://robot_description/meshes/arm1_Link.STL"/>
+        <mesh filename="$(find robot_description)/meshes/arm1_Link.STL"/>
       </geometry>
       <material name="">
@@ -115,5 +115,5 @@
       <origin xyz="0 0 0" rpy="0 0 0"/>
       <geometry>
-        <mesh filename="package://robot_description/meshes/arm1_Link.STL"/>
+        <mesh filename="$(find robot_description)/meshes/arm1_Link.STL"/>
       </geometry>
     </collision>
@@ -137,5 +137,5 @@
       <origin xyz="0 0 0" rpy="0 0 0"/>
       <geometry>
-        <mesh filename="package://robot_description/meshes/arm2_Link.STL"/>
+        <mesh filename="$(find robot_description)/meshes/arm2_Link.STL"/>
       </geometry>
       <material name="">
@@ -146,5 +146,5 @@
       <origin xyz="0 0 0" rpy="0 0 0"/>
       <geometry>
-        <mesh filename="package://robot_description/meshes/arm2_Link.STL"/>
+        <mesh filename="$(find robot_description)/meshes/arm2_Link.STL"/>
       </geometry>
     </collision>
@@ -168,5 +168,5 @@
       <origin xyz="0 0 0" rpy="0 0 0"/>
       <geometry>
-        <mesh filename="package://robot_description/meshes/arm3_Link.STL"/>
+        <mesh filename="$(find robot_description)/meshes/arm3_Link.STL"/>
       </geometry>
       <material name="">
@@ -177,5 +177,5 @@
       <origin xyz="0 0 0" rpy="0 0 0"/>
       <geometry>
-        <mesh filename="package://robot_description/meshes/arm3_Link.STL"/>
+        <mesh filename="$(find robot_description)/meshes/arm3_Link.STL"/>
       </geometry>
     </collision>
@@ -199,5 +199,5 @@
       <origin xyz="0 0 0" rpy="0 0 0"/>
       <geometry>
-        <mesh filename="package://robot_description/meshes/arm4_Link.STL"/>
+        <mesh filename="$(find robot_description)/meshes/arm4_Link.STL"/>
       </geometry>
       <material name="">
@@ -208,5 +208,5 @@
       <origin xyz="0 0 0" rpy="0 0 0"/>
       <geometry>
-        <mesh filename="package://robot_description/meshes/arm4_Link.STL"/>
+        <mesh filename="$(find robot_description)/meshes/arm4_Link.STL"/>
       </geometry>
     </collision>
@@ -230,5 +230,5 @@
       <origin xyz="0 0 0" rpy="0 0 0"/>
       <geometry>
-        <mesh filename="package://robot_description/meshes/LFs_Link.STL"/>
+        <mesh filename="$(find robot_description)/meshes/LFs_Link.STL"/>
       </geometry>
       <material name="">
@@ -239,5 +239,5 @@
       <origin xyz="0 0 0" rpy="0 0 0"/>
       <geometry>
-        <mesh filename="package://robot_description/meshes/LFs_Link.STL"/>
+        <mesh filename="$(find robot_description)/meshes/LFs_Link.STL"/>
       </geometry>
     </collision>
@@ -260,5 +260,5 @@
       <origin xyz="0 0 0" rpy="0 0 0"/>
       <geometry>
-        <mesh filename="package://robot_description/meshes/LFd_Link.STL"/>
+        <mesh filename="$(find robot_description)/meshes/LFd_Link.STL"/>
       </geometry>
       <material name="">
@@ -269,5 +269,5 @@
       <origin xyz="0 0 0" rpy="0 0 0"/>
       <geometry>
-        <mesh filename="package://robot_description/meshes/LFd_Link.STL"/>
+        <mesh filename="$(find robot_description)/meshes/LFd_Link.STL"/>
       </geometry>
     </collision>
@@ -290,5 +290,5 @@
       <origin xyz="0 0 0" rpy="0 0 0"/>
       <geometry>
-        <mesh filename="package://robot_description/meshes/LRs_Link.STL"/>
+        <mesh filename="$(find robot_description)/meshes/LRs_Link.STL"/>
       </geometry>
       <material name="">
@@ -299,5 +299,5 @@
       <origin xyz="0 0 0" rpy="0 0 0"/>
       <geometry>
-        <mesh filename="package://robot_description/meshes/LRs_Link.STL"/>
+        <mesh filename="$(find robot_description)/meshes/LRs_Link.STL"/>
       </geometry>
     </collision>
@@ -320,5 +320,5 @@
       <origin xyz="0 0 0" rpy="0 0 0"/>
       <geometry>
-        <mesh filename="package://robot_description/meshes/LRd_Link.STL"/>
+        <mesh filename="$(find robot_description)/meshes/LRd_Link.STL"/>
       </geometry>
       <material name="">
@@ -329,5 +329,5 @@
       <origin xyz="0 0 0" rpy="0 0 0"/>
       <geometry>
-        <mesh filename="package://robot_description/meshes/LRd_Link.STL"/>
+        <mesh filename="$(find robot_description)/meshes/LRd_Link.STL"/>
       </geometry>
     </collision>
@@ -350,5 +350,5 @@
       <origin xyz="0 0 0" rpy="0 0 0"/>
       <geometry>
-        <mesh filename="package://robot_description/meshes/RFs_Link.STL"/>
+        <mesh filename="$(find robot_description)/meshes/RFs_Link.STL"/>
       </geometry>
       <material name="">
@@ -359,5 +359,5 @@
       <origin xyz="0 0 0" rpy="0 0 0"/>
       <geometry>
-        <mesh filename="package://robot_description/meshes/RFs_Link.STL"/>
+        <mesh filename="$(find robot_description)/meshes/RFs_Link.STL"/>
       </geometry>
     </collision>
@@ -380,5 +380,5 @@
       <origin xyz="0 0 0" rpy="0 0 0"/>
       <geometry>
-        <mesh filename="package://robot_description/meshes/RFd_Link.STL"/>
+        <mesh filename="$(find robot_description)/meshes/RFd_Link.STL"/>
       </geometry>
       <material name="">
@@ -389,5 +389,5 @@
       <origin xyz="0 0 0" rpy="0 0 0"/>
       <geometry>
-        <mesh filename="package://robot_description/meshes/RFd_Link.STL"/>
+        <mesh filename="$(find robot_description)/meshes/RFd_Link.STL"/>
       </geometry>
     </collision>
@@ -410,5 +410,5 @@
       <origin xyz="0 0 0" rpy="0 0 0"/>
       <geometry>
-        <mesh filename="package://robot_description/meshes/RRs_Link.STL"/>
+        <mesh filename="$(find robot_description)/meshes/RRs_Link.STL"/>
       </geometry>
       <material name="">
@@ -419,5 +419,5 @@
       <origin xyz="0 0 0" rpy="0 0 0"/>
       <geometry>
-        <mesh filename="package://robot_description/meshes/RRs_Link.STL"/>
+        <mesh filename="$(find robot_description)/meshes/RRs_Link.STL"/>
       </geometry>
     </collision>
@@ -440,5 +440,5 @@
       <origin xyz="0 0 0" rpy="0 0 0"/>
       <geometry>
-        <mesh filename="package://robot_description/meshes/RRd_Link.STL"/>
+        <mesh filename="$(find robot_description)/meshes/RRd_Link.STL"/>
       </geometry>
       <material name="">
@@ -449,5 +449,5 @@
       <origin xyz="0 0 0" rpy="0 0 0"/>
       <geometry>
-        <mesh filename="package://robot_description/meshes/RRd_Link.STL"/>
+        <mesh filename="$(find robot_description)/meshes/RRd_Link.STL"/>
       </geometry>
     </collision>
