Commit message: 修改了lslidar的驱动，增加了scan_time和time_increment；建图的功能包的launch文件增加机器人direction的publisher和config文件的调整；增添了新的功能包，自动导航点抵达

File: src/robot_gazebo/urdf/robot_sim.xacro (robot description, xacro)
@@ -66,158 +66,5 @@
     <axis xyz="0 0 0"/>
   </joint>
-  <!-- arm0_link -->
-  <link name="arm0_Link">
-    <inertial>
-      <origin xyz="5.27093519414809E-05 2.44954880894475E-05 0.0113815325455051" rpy="0 0 0"/>
-      <mass value="0.469376261813121"/>
-      <inertia ixx="0.000439903649212175" ixy="6.19012321653416E-08" ixz="-2.10717922407623E-06" iyy="0.000442080302381582" iyz="-3.85248785977126E-11" izz="0.000856561950617975"/>
-    </inertial>
-    <visual>
-      <origin xyz="0 0 0" rpy="0 0 0"/>
-      <geometry>
-        <mesh filename="$(find robot_description)/meshes/arm0_Link.STL"/>
-      </geometry>
-      <material name="">
-        <color rgba="0.647058823529412 0.619607843137255 0.588235294117647 1"/>
-      </material>
-    </visual>
-    <collision>
-      <origin xyz="0 0 0" rpy="0 0 0"/>
-      <geometry>
-        <mesh filename="$(find robot_description)/meshes/arm0_Link.STL"/>
-      </geometry>
-    </collision>
-  </link>
-  <!-- arm0 joint -->
-  <joint name="arm0" type="continuous">
-    <origin xyz="0.0295174588398881 0 0.173124126705049" rpy="0 0 0"/>
-    <parent link="base_link"/>
-    <child link="arm0_Link"/>
-    <axis xyz="0 0 1"/>
-  </joint>
-  <!-- arm1_link -->
-  <link name="arm1_Link">
-    <inertial>
-      <origin xyz="-0.105007518584986 0.00141630130598419 0.0187999942153139" rpy="0 0 0"/>
-      <mass value="0.1905874165244"/>
-      <inertia ixx="4.18380122418888E-05" ixy="-8.77952273477526E-06" ixz="-1.03900484165303E-08" iyy="0.000406432980248108" iyz="1.47794609107449E-11" izz="0.000424002018340545"/>
-    </inertial>
-    <visual>
-      <origin xyz="0 0 0" rpy="0 0 0"/>
-      <geometry>
-        <mesh filename="$(find robot_description)/meshes/arm1_Link.STL"/>
-      </geometry>
-      <material name="">
-        <color rgba="0.792156862745098 0.819607843137255 0.933333333333333 1"/>
-      </material>
-    </visual>
-    <collision>
-      <origin xyz="0 0 0" rpy="0 0 0"/>
-      <geometry>
-        <mesh filename="$(find robot_description)/meshes/arm1_Link.STL"/>
-      </geometry>
-    </collision>
-  </link>
-  <!-- arm1 joint -->
-  <joint name="arm1" type="revolute">
-    <origin xyz="0.02 0.0183 0.0595" rpy="1.5708 0 0"/>
-    <parent link="arm0_Link"/>
-    <child link="arm1_Link"/>
-    <axis xyz="0 0 1"/>
-    <limit lower="-210" upper="0" effort="1" velocity="3"/>
-  </joint>
-  <!-- arm2_link -->
-  <link name="arm2_Link">
-    <inertial>
-      <origin xyz="0.100452932197325 0.0447481861533194 -0.0181893769189027" rpy="0 0 0"/>
-      <mass value="0.164248712945774"/>
-      <inertia ixx="3.52887905356114E-05" ixy="-2.00181663560874E-05" ixz="5.21115865733209E-09" iyy="0.00029554091042407" iyz="-3.44733343118317E-10" izz="0.000308884693204529"/>
-    </inertial>
-    <visual>
-      <origin xyz="0 0 0" rpy="0 0 0"/>
-      <geometry>
-        <mesh filename="$(find robot_description)/meshes/arm2_Link.STL"/>
-      </geometry>
-      <material name="">
-        <color rgba="1 1 1 1"/>
-      </material>
-    </visual>
-    <collision>
-      <origin xyz="0 0 0" rpy="0 0 0"/>
-      <geometry>
-        <mesh filename="$(find robot_description)/meshes/arm2_Link.STL"/>
-      </geometry>
-    </collision>
-  </link>
-  <!-- arm2 joint -->
-  <joint name="arm2" type="revolute">
-    <origin xyz="-0.214299994813131 0 0.0376000028997485" rpy="0 0 0"/>
-    <parent link="arm1_Link"/>
-    <child link="arm2_Link"/>
-    <axis xyz="0 0 -1"/>
-    <limit lower="0" upper="270" effort="1" velocity="3"/>
-  </joint>
-  <!-- arm3_link -->
-  <link name="arm3_Link">
-    <inertial>
-      <origin xyz="0.0244536421910909 -0.0093611713162593 -0.0184330992425119" rpy="0 0 0"/>
-      <mass value="0.0312238812156817"/>
-      <inertia ixx="1.2997419944031E-05" ixy="-6.86664871709515E-07" ixz="-9.49084586365268E-09" iyy="1.14173396064683E-05" iyz="4.27514678311462E-09" izz="1.1219689644564E-05"/>
-    </inertial>
-    <visual>
-      <origin xyz="0 0 0" rpy="0 0 0"/>
-      <geometry>
-        <mesh filename="$(find robot_description)/meshes/arm3_Link.STL"/>
-      </geometry>
-      <material name="">
-        <color rgba="1 1 1 1"/>
-      </material>
-    </visual>
-    <collision>
-      <origin xyz="0 0 0" rpy="0 0 0"/>
-      <geometry>
-        <mesh filename="$(find robot_description)/meshes/arm3_Link.STL"/>
-      </geometry>
-    </collision>
-  </link>
-  <!-- arm3 joint -->
-  <joint name="arm3" type="revolute">
-    <origin xyz="0.195198405547995 0.0479983915101106 0.000499985962073995" rpy="0.00872697851439958 -0.00872598171315928 -7.61524215215586E-05"/>
-    <parent link="arm2_Link"/>
-    <child link="arm3_Link"/>
-    <axis xyz="-0.00872587097686232 -0.00872653549837341 -0.99992385047757"/>
-    <limit lower="0" upper="100" effort="1" velocity="3"/>
-  </joint>
-  <!-- arm4_link -->
-  <link name="arm4_Link">
-    <inertial>
-      <origin xyz="0.0347390678915086 -0.00413801569158295 -0.0209305905705711" rpy="0 0 0"/>
-      <mass value="0.0522475609584348"/>
-      <inertia ixx="1.36823938394385E-05" ixy="2.66574817985518E-06" ixz="8.39394854007867E-07" iyy="9.79309028256577E-06" iyz="-1.69593151918628E-06" izz="1.75606392336261E-05"/>
-    </inertial>
-    <visual>
-      <origin xyz="0 0 0" rpy="0 0 0"/>
-      <geometry>
-        <mesh filename="$(find robot_description)/meshes/arm4_Link.STL"/>
-      </geometry>
-      <material name="">
-        <color rgba="0.650980392156863 0.619607843137255 0.588235294117647 1"/>
-      </material>
-    </visual>
-    <collision>
-      <origin xyz="0 0 0" rpy="0 0 0"/>
-      <geometry>
-        <mesh filename="$(find robot_description)/meshes/arm4_Link.STL"/>
-      </geometry>
-    </collision>
-  </link>
-  <!-- arm4 joint -->
-  <joint name="arm4" type="revolute">
-    <origin xyz="0.0398926340613602 -0.0346685199789408 -0.0183469477877459" rpy="1.56824861064815 0.00509594419856987 -0.366478515653153"/>
-    <parent link="arm3_Link"/>
-    <child link="arm4_Link"/>
-    <axis xyz="-0.00872587097688493 -0.00872653523448956 -0.999923850479873"/>
-    <limit lower="-90" upper="90" effort="1" velocity="3"/>
-  </joint>
+  <!-- ===== ARM LINKS & JOINTS REMOVED (restore from git history if needed) ===== -->
   <!-- LFs link (左前 steering) -->
   <link name="LFs_Link">
@@ -565,50 +412,5 @@
     </collision>
   </gazebo>
-  <!-- Arm links: disable collision (not simulated) -->
-  <gazebo reference="arm0_Link">
-    <collision>
-      <geometry>
-        <box>
-          <size>0.01 0.01 0.01</size>
-        </box>
-      </geometry>
-    </collision>
-  </gazebo>
-  <gazebo reference="arm1_Link">
-    <collision>
-      <geometry>
-        <box>
-          <size>0.01 0.01 0.01</size>
-        </box>
-      </geometry>
-    </collision>
-  </gazebo>
-  <gazebo reference="arm2_Link">
-    <collision>
-      <geometry>
-        <box>
-          <size>0.01 0.01 0.01</size>
-        </box>
-      </geometry>
-    </collision>
-  </gazebo>
-  <gazebo reference="arm3_Link">
-    <collision>
-      <geometry>
-        <box>
-          <size>0.01 0.01 0.01</size>
-        </box>
-      </geometry>
-    </collision>
-  </gazebo>
-  <gazebo reference="arm4_Link">
-    <collision>
-      <geometry>
-        <box>
-          <size>0.01 0.01 0.01</size>
-        </box>
-      </geometry>
-    </collision>
-  </gazebo>
+  <!-- Arm links: removed with arm definition above -->
   <!-- ===== Planar Move Plugin (cmd_vel → base motion + odom) ===== -->
   <gazebo>
